File: PCB/hacropad.kicad_pcb (KiCad board)
At the start: 2 copper layers, 35 parts, among them SW1 SW_Push, SW10 SW_Push, SW2 SW_Push, SW3 SW_Push, SW4 SW_Push, SW5 SW_Push, SW6 SW_Push, SW7 SW_Push, SW8 SW_Push, SW9 SW_Push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

Commit message: Add files via upload
Other:
- board text added: "............ ...............:::::---... .................:-++**#*+=-=+====--:... ....:-=+++==+++=+#%@@*-%@@#*#%#----:-:.. ....+***#######++=:-+==+%@++@#==@%-+*+*%#*=----:.. ...+%%%%%%%%%%###*+=+++=+*%@@##%@***=#%**#%@#=----:.. ...**%%%#%#####****+++++*%##%%@@*+++++=+*#%@%*=----:. ..-**#%#%********++++++++%@@@@@@#+++++++%@@@@@#-----... .-..-###%***++++++=++=++**####%@@#*++*@@@%%%%%=-----.. .....+#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"
- board text added: "Can I have some...?"
- board text added: "Great baking"
- board text added: "The Hacropad By KIS"
- board text added: "Well well well it looks like you know how a screwdriver works."
- board text added: "XIAO HERE!"
- board text added: "YOLO!!"
Changed lines of the file:
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@@
 		(layer "B.Cu")
+	)
+	(gr_text "Well well well it looks\nlike you know how a\nscrewdriver works."
+		(at 157.89 95.84 0)
+		(layer "F.Cu")
+		(effects
+			(font
+				(size 1.5 1.5)
+				(thickness 0.3)
+				(bold yes)
+			)
+			(justify left bottom)
+		)
+	)
+	(gr_text "XIAO HERE!"
+		(at 141.25 37.53 0)
+		(layer "F.Cu")
+		(effects
+			(font
+				(size 1.5 1.5)
+				(thickness 0.3)
+				(bold yes)
+			)
+			(justify left bottom)
+		)
+	)
+	(gr_text "YOLO!!"
+		(at 116.74 86.64 0)
+		(layer "F.Cu")
+		(effects
+			(font
+				(size 1.5 1.5)
+				(thickness 0.3)
+				(bold yes)
+			)
+			(justify left bottom)
+		)
+	)
+	(gr_text "The Hacropad\nBy KIS"
+		(at 113.37 28.87 0)
+		(layer "F.Cu")
+		(effects
+			(font
+				(size 1.5 1.5)
+				(thickness 0.3)
+				(bold yes)
+			)
+			(justify left bottom)
+		)
+	)
+	(gr_text "Can I have some...?"
+		(at 112.91 116.38 180)
+		(layer "B.Cu")
+		(effects
+			(font
+				(size 1.5 1.5)
+				(thickness 0.3)
+				(bold yes)
+			)
+			(justify left bottom mirror)
+		)
+	)
+	(gr_text "Great baking"
+		(at 112.69 119.49 180)
+		(layer "B.Cu")
+		(effects
+			(font
+				(size 1.5 1.5)
+				(thickness 0.3)
+				(bold yes)
+			)
+			(justify left bottom mirror)
+		)
+	)
+	(gr_text "                                                         \n                                                         \n                                    ............         \n                       ...............:::::---...        \n           .................:-++**#*+=-=+====--:...      \n           ....:-=+++==+++=+#%@@*-%@@#*#%#----:-:..      \n  ....+***#######++=:-+==+%@++@#==@%-+*+*%#*=----:..     \n...+%%%%%%%%%%###*+=+++=+*%@@##%@***=#%**#%@#=----:..    \n...**%%%#%#####****+++++*%##%%@@*+++++=+*#%@%*=----:.    \n..-**#%#%********++++++++%@@@@@@#+++++++%@@@@@#-----...  \n .-..-###%***++++++=++=++**####%@@#*++*@@@%%%%%=-----..  \n .....+#%*#**+++++++++++=++#@@@@@%@@@%%@%%%@@%======--.  \n     .:*%%#*******+++++***+=+**#%@@@@#@@@#@@#====--==+:  \n     ..-*%%#*#########*+=-+***++**##*#%%#*#*********+=.  \n      ..+#%%##########*+==-:-=+******############*-:...  \n       ..##%%*#########******###%#%%%%%%%%%%%%%%#*-:.    \n        .-##%#*#####%%%%%%%%%%%%%%%%%%%%%@%##-:....      \n        ..+++*#%%%%%%%%%%%%%@%%@%%##%%%%%#*:::...        \n        ...#***%%%%@@@%@@@@@@%%%#**+=-::.........        \n        ...:***#=-:.:+=-#*==-:::.............            \n        ....-*==-............................            \n           ..=-...     ..                                \n            ..:...                                       \n             ...                                         "
+		(at 184.65 45.57 0)
+		(layer "B.Cu")
+		(effects
+			(font
+				(size 0.6 0.6)
+				(thickness 0.15)
+			)
+			(justify left bottom mirror)
+		)
 	)
 	(segment

Commit message: Add files via upload
Routing:
- net fIVER: track 259.7 -> 303.4 mm
- net Floor: track 241.3 -> 275.5 mm
Other:
- board outline added: 74.4 x 99.2 mm
Changed lines of the file:
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@@
 		(stroke
 			(width 0.2)
-			(type default)
+			(type solid)
 		)
 		(fill no)
-		(layer "B.Cu")
+		(layer "Edge.Cuts")
 	)
 	(gr_text "Well well well it looks\nlike you know how a\nscrewdriver works."
@@
 	)
 	(segment
+		(start 179 46.27)
+		(end 179 29)
+		(width 0.2)
+		(layer "F.Cu")
+		(net 22)
+	)
+	(segment
 		(start 154.274 85.411)
 		(end 154.974 86.111)
@@
 	)
 	(segment
+		(start 177.34 47.93)
+		(end 179 46.27)
+		(width 0.2)
+		(layer "F.Cu")
+		(net 22)
+	)
+	(segment
 		(start 138.74 85.01)
 		(end 139.141 85.411)
@@
 	)
 	(segment
+		(start 179 29)
+		(end 176.4685 26.4685)
+		(width 0.2)
+		(layer "F.Cu")
+		(net 22)
+	)
+	(segment
+		(start 176.4685 26.4685)
+		(end 155.915 26.4685)
+		(width 0.2)
+		(layer "F.Cu")
+		(net 22)
+	)
+	(segment
 		(start 170.385657 67.614343)
 		(end 169.392314 66.621)
@@
 	)
 	(segment
+		(start 175.59 44.43)
+		(end 175.59 30.59)
+		(width 0.2)
+		(layer "F.Cu")
+		(net 23)
+	)
+	(segment
 		(start 130.602314 66.231)
 		(end 120.221 66.231)
@@
 	)
 	(segment
+		(start 174 29)
+		(end 173.9915 29.0085)
+		(width 0.2)
+		(layer "F.Cu")
+		(net 23)
+	)
+	(segment
+		(start 175.59 30.59)
+		(end 174 29)
+		(width 0.2)
+		(layer "F.Cu")
+		(net 23)
+	)
+	(segment
 		(start 175.35 78.76)
 		(end 175.35 78.62)
@@
 		(width 0.2)
 		(layer "F.Cu")
+		(net 23)
+	)
+	(segment
+		(start 173.9915 29.0085)
+		(end 155.915 29.0085)
+		(width 0.2)
+		(layer "F.Cu")
